File: Reel/Reel.kicad_sch (KiCad schematic)
At the start: 10 parts, among them J1 USB_C_Receptacle_USB2.0, U3 XC6210B332MR-G, U4 USBLC6-2P6

Commit message: update
Parts:
- removed D2: B5817, Diode_SMD:D_SOD-323, symbol Device:D_Schottky
- removed FB1: FerriteBead_Small, Inductor_SMD:L_0603_1608Metric, symbol Device:FerriteBead_Small
- removed U3: XC6210B332MR-G, Package_TO_SOT_SMD:SOT-23-5, symbol Regulator_Linear:AP2127K-3.3
- removed U4: USBLC6-2P6, Package_TO_SOT_SMD:SOT-666, symbol Power_Protection:USBLC6-2P6
- added U1: RT9013-33GB, Package_TO_SOT_SMD:SOT-23-5, symbol rp-micro:RT9013-33GB
- added U2: SRV05-4, Package_TO_SOT_SMD:SOT-23-6, symbol Power_Protection:SRV05-4
- C1, C2: value 1µ -> 1uF; footprint Capacitor_SMD:C_0603_1608Metric -> Capacitor_SMD:C_0402_1005Metric; LCSC C19666 -> C52923
- F1: value Polyfuse -> 500mA, 6V; footprint Fuse:Fuse_0603_1608Metric -> Fuse:Fuse_0805_2012Metric; LCSC C69679 -> C269104
Connections:
- net +3V3: now also U1.5 (VOUT)
- net +5V: now also F1.2, U1.1 (VIN), U1.3 (EN), U2.5 (VP)
- net GND: now also J1.S1 (SHIELD), U1.2 (GND), U2.2 (VN)
- net USB_D+: now also U2.6 (IO4)
- net USB_D-: now also U2.1 (IO1)
- no-connect marks 2 -> 4
Other:
- moved on the sheet: C2, F1
