File: Reel/RP2040.kicad_sch (KiCad schematic)
At the start: 32 parts, among them J105 NA_Conn_01x04_Female, SW1 BOOT, SW2 RESET, U3 W25Q128JVS, U4 RP2040, Y1 12MHz

Commit message: update
Parts:
- removed R10: 5.1k, Resistor_SMD:R_0402_1005Metric, symbol Device:R
- removed R11: 10k, Resistor_SMD:R_0402_1005Metric, symbol Device:R
- C10, C11, C12, C13, C14, C15, C16: LCSC C1525 -> C307331
- C3: renamed from C19; LCSC C1525 -> C307331
- C4: renamed from C3; value 15pF -> 20pF; LCSC C1548 -> C1554
- C5: renamed from C4; value 15pF -> 20pF; LCSC C1548 -> C1554
- C8: renamed from C7; LCSC C1525 -> C307331
- C9: renamed from C8; LCSC C1525 -> C307331
- R3: footprint Resistor_SMD:R_0402_1005Metric -> Resistor_SMD:R_0603_1608Metric; LCSC C25100 -> C25190
- R4: renamed from R6; footprint Resistor_SMD:R_0402_1005Metric -> Resistor_SMD:R_0603_1608Metric; LCSC C25100 -> C25190
- R5015: LCSC C105875 -> C11702
- U3: LCSC C190862 -> C97521
- renumbered R4 to R5, R5 to R6, R9 to R7, R10 to R8
Connections:
- net at C4.2, U4.20 (XIN): now also Y1.3; no longer Y1.1
- net at C5.2, R7.1: now also Y1.1; no longer Y1.3
- net VBUS_DET: no longer names the net of U4.30 (GPIO19)
- no-connect marks 12 -> 13
Other:
- moved on the sheet: C3, R5, R6, U3, Y1

Commit message: multi layout
Parts:
- removed C5015: 1uF, Capacitor_SMD:C_0402_1005Metric, symbol Device:C
- removed D3 (x2): SK6812, local-libraries:SK6812-MINI-E, symbol sk6805-ec15:SK6805-EC15
- removed R5015: 330, Resistor_SMD:R_0402_1005Metric, symbol Device:R
Connections:
- net DIN: no longer names the net of U4.2 (GPIO0)
