File: Reel/Reel.kicad_pcb (KiCad board)
At the start: 2 copper layers, 275.9 x 93.2 mm, 134 parts, among them J1 USB_C_Receptacle_USB2.0, J2 NA_Conn_01x04_Female, SW1 BOOT, SW2 RESET, U1 XC6210B332MR-G, U2 USBLC6-2P6, U3 W25Q128JVS, U4 RP2040, Y1 12MHz

Commit message: update
Parts:
- removed C19: 100nF, Capacitor_SMD:C_0402_1005Metric
- removed D1001: B5817, Diode_SMD:D_SOD-323
- removed FB1: FerriteBead_Small, Inductor_SMD:L_0603_1608Metric
- removed R10: 10k, Resistor_SMD:R_0402_1005Metric
- removed R11: 330, Resistor_SMD:R_0402_1005Metric
- added C9: 100nF, Capacitor_SMD:C_0402_1005Metric, B.Cu at (140.5, 84.9)
- C1, C2: value 1µ -> 1uF; footprint Capacitor_SMD:C_0603_1608Metric -> Capacitor_SMD:C_0402_1005Metric
- C3: value 15pF -> 100nF
- C4: value 15pF -> 20pF
- C5: value 1uF -> 20pF
- C7: value 100nF -> 1uF
- F1: value Polyfuse -> 500mA, 6V; footprint Fuse:Fuse_0603_1608Metric -> Fuse:Fuse_0805_2012Metric
- R3: footprint Resistor_SMD:R_0402_1005Metric -> Resistor_SMD:R_0603_1608Metric
- R4: value 1k -> 27; footprint Resistor_SMD:R_0402_1005Metric -> Resistor_SMD:R_0603_1608Metric
- R5: value 10k -> 1k
- R6: value 27 -> 10k
- R7: value 5.1k -> 1k
- R9: value 1k -> 330
- U1: value XC6210B332MR-G -> RT9013-33GB
- U2: value USBLC6-2P6 -> SRV05-4; footprint Package_TO_SOT_SMD:SOT-666 -> Package_TO_SOT_SMD:SOT-23-6
- moved C3 28.5 mm to (134.9, 58.4), turned to 180 degrees
- moved C2 19.2 mm to (44.4, 56.6), turned to 90 degrees
- moved U1 16.3 mm to (41.6, 55.8), turned to 0 degrees
- moved R6 13.8 mm to (146.3, 58.4)
- moved C7 13.8 mm to (138.6, 71.3), turned to 90 degrees
- moved C5 13.4 mm to (142.9, 85.7), turned to 90 degrees
- moved R4 12.3 mm to (140.1, 70.7)
- moved R9 10.6 mm to (148.4, 74.8), turned to 0 degrees
- moved R7 8.89 mm to (142.9, 83.7)
- moved U2 5.80 mm to (31.8, 50.8), turned to 0 degrees
- moved C1 5.74 mm to (40.5, 53.4), turned to 0 degrees
- moved R8 4.96 mm to (139.3, 84.9), turned to 90 degrees
- moved C4 4.90 mm to (147.3, 84.1)
- moved R5 4.29 mm to (146.6, 56.4), turned to 0 degrees
- moved U3 2.85 mm to (140.8, 60.8)
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Connections:
- C3 pad 1: GND -> +3V3
- C3 pad 2: Net-(U4-XIN) -> GND
- C4 pad 2: Net-(C4-Pad2) -> Net-(U4-XIN)
- C5 pad 1: +3V3 -> GND
- C5 pad 2: GND -> Net-(C5-Pad2)
- C6 pad 1: +1V1 -> +3V3
- F1 pad 2: Net-(D1001-A) -> +5V
- J1 pad S1: Net-(J1-SHIELD) -> GND
- R4 pad 1: /RP2040/BOOT -> /USB_D-
- R4 pad 2: /RP2040/QSPI_SS -> Net-(U4-USB_DM)
- R5 pad 1: +3V3 -> /RP2040/BOOT
- R6 pad 1: /USB_D- -> +3V3
- R6 pad 2: Net-(U4-USB_DM) -> /RP2040/QSPI_SS
- R7 pad 1: /RP2040/VBUS_DET -> Net-(C5-Pad2)
- R7 pad 2: VBUS -> Net-(U4-XOUT)
- R8 pad 1: GND -> +3V3
- R8 pad 2: /RP2040/VBUS_DET -> /RP2040/~{RESET}
- R9 pad 1: Net-(C4-Pad2) -> DIN
- R9 pad 2: Net-(U4-XOUT) -> Net-(LED1-DIN)
- U2 pad 3: /USB_D+ -> unconnected-(U2-IO2-Pad3)
- U2 pad 4: /USB_D+ -> unconnected-(U2-IO3-Pad4)
- U2 pad 5: VBUS -> +5V
- U2 pad 6: /USB_D- -> /USB_D+
- U4 pad 30: /RP2040/VBUS_DET -> unconnected-(U4-GPIO19-Pad30)
- Y1 pad 1: Net-(U4-XIN) -> Net-(C5-Pad2)
- Y1 pad 3: Net-(C4-Pad2) -> Net-(U4-XIN)
Routing:
- net VBUS: track 145.9 -> 10.9 mm, vias 6 -> 0
- net +3V3: track 398.0 -> 365.3 mm, vias 7 -> 8
- net Net-(J1-SHIELD): track 21.1 -> 0.00 mm
- net GND: track 57.1 -> 68.1 mm, vias 63 -> 54
- net /RP2040/VBUS_DET: track 6.08 -> 0.00 mm
- net /RP2040/QSPI_SS: track 17.5 -> 22.2 mm
- net Net-(J1-CC2): track 2.51 -> 7.09 mm, vias 0 -> 2
- net /RP2040/QSPI_D3: track 20.0 -> 24.0 mm
- net /RP2040/QSPI_D0: track 15.3 -> 19.2 mm
- net /RP2040/QSPI_SCLK: track 18.6 -> 22.3 mm
- net Net-(D1001-A): track 3.63 -> 0.00 mm
- net +5V: track 16.4 -> 19.7 mm, vias 2 -> 0
- net /RP2040/QSPI_D1: track 12.8 -> 16.0 mm
- net Net-(C4-Pad2): track 2.84 -> 0.00 mm
- net /RP2040/QSPI_D2: track 11.8 -> 14.6 mm
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
Commit message: multi layout
Parts:
- removed C17: 1uF, Capacitor_SMD:C_0402_1005Metric
- removed LED1, LED2: SK6812, local-libraries:SK6812-MINI-E
- removed R9: 330, Resistor_SMD:R_0402_1005Metric
- added D47: 1N4148, Diode_SMD:D_SOD-123, B.Cu at (261.0, 111.6)
- added KEY47: SW_Push_45deg, MX_Solderable:MX-Solderable-1U, F.Cu at (252.5, 107.1)
- added KEY48: SW_Push_45deg, MX_Solderable:MX-Solderable-1.25U, F.Cu at (248.0, 107.1)
- locked (x2): footprint MX_Solderable:MX-Solderable-1.25U -> MX_Solderable:MX-Solderable-1U
- moved locked 14.5 mm to (233.4, 107.1)
- moved D45 14.1 mm to (239.3, 111.9)
- moved J1 1.37 mm to (31.8, 35.9)
- moved C14 1.11 mm to (147.4, 74.0), turned to 90 degrees
- moved R1 1.02 mm to (30.3, 43.1)
- moved R2 0.60 mm to (35.6, 43.5)
- moved F1 0.30 mm to (33.7, 45.7)
- moved locked 0.15 mm to (271.6, 107.1)
Connections:
- U4 pad 2: DIN -> unconnected-(U4-GPIO0-Pad2)
Routing:
- net +3V3: track 365.3 -> 197.7 mm, vias 8 -> 5
- net Net-(LED1-DIN): track 161.3 -> 0.00 mm, vias 2 -> 0
- net COL_11: track 150.0 -> 194.4 mm
- net Net-(D47-A): track 0.00 -> 28.0 mm
- net Net-(LED1-DOUT): track 13.1 -> 0.00 mm
- net COL_10: track 166.8 -> 161.3 mm
- net DIN: track 2.61 -> 0.00 mm
- net COL_8: track 123.7 -> 121.3 mm
- net /USB_D-: track 134.4 -> 136.5 mm
- net GND: track 68.1 -> 66.1 mm, vias 54 -> 49
- net Net-(J1-CC2): track 7.09 -> 5.13 mm
- net /USB_D+: track 136.0 -> 137.5 mm
- net VBUS: track 10.9 -> 12.4 mm
- net Net-(D45-A): track 12.8 -> 11.4 mm
Other:
- board size 275.9 x 93.2 mm -> 270.4 x 92.5 mm
