File: Reel/key_matrix.kicad_sch (KiCad schematic)
At the start: 92 parts

Commit message: multi layout
Parts:
- added D47: 1N4148, Diode_SMD:D_SOD-123, symbol Diode:1N4148
- added KEY47: SW_Push_45deg, MX_Solderable:MX-Solderable-1U, symbol Switch:SW_Push_45deg
- added KEY48: SW_Push_45deg, MX_Solderable:MX-Solderable-1.25U, symbol Switch:SW_Push_45deg
- KEY45, KEY46: footprint MX_Solderable:MX-Solderable-1.25U -> MX_Solderable:MX-Solderable-1U
Connections:
- net COL_11: now also KEY47.1, KEY48.1
- net ROW_3: now also D47.1 (K)
- new net: D47.2 (A), KEY47.2, KEY48.2
Other:
- moved on the sheet: D13, D25, D38, D46, KEY13, KEY25, KEY38, KEY46
